File: rl78prog/KiCAD/FTDI231XS/SerialUSB.kicad_pcb (KiCad board)
At the start: 2 copper layers, 23 parts, among them P1 USB_OTG, P2 CONN_02X05, P3 CONN_02X03, SW1 3P-SW, U1 NJU7223DL1-33, U2 FT231XS

Commit message: update
Parts:
- P1: footprint Connect:USB_Micro-B -> Akizuki:HRS-MICRO-USB-B
- moved C2 7.63 mm to (110.5, 111.8), turned to 0 degrees
- moved C1 7.37 mm to (110.5, 117.9), turned to 180 degrees
- moved R3 7.01 mm to (152.6, 125.7)
- moved R4 7.01 mm to (152.6, 104.1)
- moved C7 6.80 mm to (117.2, 125.0)
- moved R5 6.18 mm to (110.5, 121.4)
- moved D1 5.00 mm to (160.0, 125.0)
- moved D2 5.00 mm to (160.0, 105.0)
- moved D3 5.00 mm to (110.0, 125.0)
- moved R1 2.45 mm to (110.7, 113.8)
- moved R2 2.20 mm to (110.7, 115.8)
- moved FB1 1.92 mm to (110.7, 107.8)
- moved P1 1.64 mm to (102.5, 115.0), turned to 90 degrees
- moved C8 1.34 mm to (141.1, 105.8)
- moved C6 0.54 mm to (138.2, 105.8)
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Routing:
- net Net-(C2-Pad1): track 0.00 -> 6.67 mm
- net Net-(C1-Pad2): track 0.00 -> 6.24 mm
- net Net-(R2-Pad1): track 0.00 -> 5.16 mm
- net Net-(R1-Pad1): track 0.00 -> 3.48 mm
Other:
- board outline added: 66.5 x 26.5 mm
